File: DCP2PLS.brd (EAGLE design)
At the start: 20 x 16 mm, 2 parts, among them CON4 CON-6P, CON6 PINHEAD_1X06-2.54

Commit message: updates
Parts:
- moved CON4 2.55 mm to (7.00, 0.00)
- moved CON6 2.55 mm to (-8.00, 0.00)
Routing:
- added copper zone on layer 16, net G
Other:
- outline, holes or cut-outs redrawn
